File: doc/circuits/decoder.kicad_sch (KiCad schematic)
At the start: 11 parts, among them U1 74LS138, U10 74LS161, U11 74LS161, U2 74LS161, U3 74LS04, U4 74LS08, U5 74LS04, U6 74LS161, U7 74LS161, U8 74LS161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

Commit message: Built circuits in Kicad to be used in documentation later
Other:
- note added: "MC 0-3"
- note added: "MC 4-7"
- note added: "MICROCODE DECODER"
- note removed: "Bank Select"
- note removed: "Data 0-3"
- note removed: "Data 4-7"
- note removed: "Decoder"
- note removed: "Master clock"
- note removed: "The clock divider takes the master clock (M_CLK) and subdivides it into 4 clocks, the last of which is sent to all other modules (CLK). The first 3 clocks are used to sequentially load in the control signals from the microcode ROM (not included), which is addressed by the instruction register and bank index."
- note removed: "To other modules"
Changed lines of the file:
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@@
     (fill (type none))
-  )
-  (text "The clock divider takes the master clock (M_CLK) and subdivides it into 4 clocks, the last of which is \nsent to all other modules (CLK). The first 3 clocks are used to sequentially load in the control signals \nfrom the microcode ROM (not included), which is addressed by the instruction register and bank index."
-    (at 180.34 176.53 0)
-    (effects (font (size 1.27 1.27)) (justify left bottom))
   )
   (text "BANK 0" (at 256.54 101.6 0)
     (effects (font (size 3 3)) (justify left bottom))
   )
-  (text "Data 4-7" (at 22.86 111.76 0)
-    (effects (font (size 1.27 1.27)) (justify left bottom))
-  )
-  (text "Data 4-7" (at 208.28 24.13 90)
+  (text "MC 4-7" (at 22.86 107.95 0)
     (effects (font (size 1.27 1.27)) (justify left bottom))
   )
@@
     (effects (font (size 3 3)) (justify left bottom))
   )
-  (text "To other modules" (at 25.4 24.13 0)
-    (effects (font (size 1.27 1.27)) (justify left bottom))
-  )
-  (text "Master clock" (at 27.94 52.07 0)
-    (effects (font (size 1.27 1.27)) (justify left bottom))
-  )
   (text "BANK 2" (at 26.67 160.02 0)
     (effects (font (size 3 3)) (justify left bottom))
   )
-  (text "Data 0-3" (at 22.86 102.87 0)
-    (effects (font (size 1.27 1.27)) (justify left bottom))
-  )
-  (text "Data 0-3" (at 200.66 24.13 90)
-    (effects (font (size 1.27 1.27)) (justify left bottom))
-  )
-  (text "Bank Select" (at 25.4 30.48 0)
+  (text "MC 0-3" (at 22.86 104.14 0)
     (effects (font (size 1.27 1.27)) (justify left bottom))
   )
@@
     (effects (font (size 3 3)) (justify left bottom))
   )
-  (text "Decoder" (at 189.23 190.5 0)
-    (effects (font (size 1.27 1.27)) (justify left bottom))
+  (text "MICROCODE DECODER" (at 205.74 176.53 0)
+    (effects (font (size 3 3)) (justify left bottom))
   )
   (global_label "CR" (shape output) (at 134.62 179.07 270) (fields_autoplaced)
