File: doc/circuits/signal_distributor.kicad_sch (KiCad schematic)
At the start: 12 parts, among them U1 74LS138, U10 74LS161, U11 74LS161, U12 74LS04, U2 74LS161, U3 74LS04, U4 74LS08, U5 74LS04, U6 74LS161, U7 74LS161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

Commit message: More documentation done
Other:
- note added: "CONTROL UNIT 2"
- note removed: "CONTROL SIGNAL DISTRIBUTOR"

Commit message: worked on docs a bit
Other:
- company: (none) -> J. Heit
Changed lines of the file:
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@@
 	(generator_version "8.0")
 	(paper "A4")
+	(title_block
+		(date "2025")
+		(rev "1")
+		(company "J. Heit")
+	)
 	(junction
 		(at 140.97 33.02)
@@
 		)
 		(property "Value" "74LS161"
-			(at 82.55 148.59 90)
+			(at 82.55 144.272 90)
 			(effects
 				(font
@@
 		(on_board yes)
 		(dnp no)
-		(fields_autoplaced yes)
 		(property "Reference" "U10"
 			(at 230.5619 71.12 90)
@@
 		)
 		(property "Value" "74LS161"
-			(at 233.1019 71.12 90)
+			(at 240.792 99.568 0)
 			(effects
 				(font
 					(size 1.27 1.27)
 				)
-				(hide yes)
 			)
 		)
@@
 		)
 		(property "Value" "74LS161"
-			(at 35.56 148.59 90)
+			(at 36.068 144.018 90)
 			(effects
 				(font
@@
 		)
 		(property "Value" "74LS161"
-			(at 177.8 148.59 90)
+			(at 177.292 144.018 90)
 			(effects
 				(font
@@
 		)
 		(property "Value" "74LS161"
-			(at 130.81 148.59 90)
+			(at 130.302 144.018 90)
 			(effects
 				(font
@@
 		)
 		(property "Value" "74LS161"
-			(at 240.03 50.8 0)
+			(at 240.538 51.816 0)
 			(effects
 				(font
