File: doc/circuits/signal_fetcher.kicad_sch (KiCad schematic)
At the start: 11 parts, among them U1 28C64, U10 74LS04, U11 74LS173, U2 74LS157, U3 74LS173, U4 74LS173, U5 74LS04, U6 28C64, U7 74LS163, U8 74LS14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

Commit message: More documentation done
Connections:
- net GND: no longer U11.7 (Cp), U3.10 (E2), U3.7 (Cp), U4.10 (E2), U4.7 (Cp), U5.2, U8.1
- new net: U3.10 (E2), U4.10 (E2), U5.2
- new net CLK: U11.7 (Cp), U3.7 (Cp), U4.7 (Cp), U8.1
Other:
- note added: "CONTROL UNIT 1"
- note removed: "CONTROL SIGNAL FETCHER"

Commit message: worked on docs a bit
Other:
- company: (none) -> J. Heit
Changed lines of the file:
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@@
 	(generator_version "8.0")
 	(paper "A4")
+	(title_block
+		(date "2025")
+		(rev "1")
+		(company "J. Heit")
+	)
 	(junction
 		(at 209.55 64.77)
