File: doc/circuits/ram.kicad_sch (KiCad schematic)
At the start: 12 parts, among them U1 AS6C4008-55PCN, U10 74LS04, U11 74LS08, U12 74LS04, U2 AS6C4008-55PCN, U3 74HC245, U4 74HC245, U5 74LS04, U6 74HC86, U7 74HC86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

Commit message: Updated schematics
Connections:
- net OE_RAM: now also U8.2; no longer U8.1
- net WE_RAM: now also U8.1; no longer U8.2
Other:
- note removed: "Address Bus"
- note removed: "Databus 0-7"
- note removed: "Databus 8-15"

Commit message: more documentation
Connections:
- net CLK renamed M_CLK
Other:
- note added: "NOTE: Logic is needed to be able to intercept the output and show this on a LED array, while not making the data available on the bus."
- note removed: "NOTE: Logic is needed to be able to intercept the output and show this on an LED array, while not making the data available on the bus."
