File: doc/circuits/loop_skip_register.kicad_sch (KiCad schematic)
At the start: 12 parts, among them U1 74LS193, U10 74LS32, U11 74LS32, U12 74LS04, U13 74LS193, U3 74LS245, U4 74LS04, U5 74LS04, U6 74LS32, U7 74LS245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

Commit message: Updated schematics
Parts:
- removed U12, U4, U5: 74LS04, symbol 74xx:74LS04
- removed U3, U7: 74LS245, symbol 74xx:74LS245
Connections:
- net +5V: now also U1.11 (~{LOAD}), U13.11 (~{LOAD})
- net at U1.3 (QA): now also U6.1; no longer U9.5
- net at U1.2 (QB): now also U6.2; no longer U9.4
- net at U1.6 (QC): now also U6.4; no longer U9.2
- net at U1.7 (QD): now also U6.5; no longer U9.1
- net at U13.3 (QA): now also U9.1; no longer U6.5
- net at U13.2 (QB): now also U9.2; no longer U6.4
- net at U13.6 (QC): now also U9.4; no longer U6.2
- net at U13.7 (QD): now also U9.5; no longer U6.1
- net S: now reaches U11.3
- no-connect marks 2 -> 10
Other:
- note added: "LS-REGISTER MODULE"
- note removed: "D-REGISTER MODULE"

Commit message: documentation
Connections:
- net D_D renamed D_LS
- net U_D renamed U_LS
Changed lines of the file:
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@@
 		)
 	)
-	(global_label "U_D"
+	(global_label "U_LS"
 		(shape input)
 		(at 63.5 120.65 180)
@@
 		)
 		(property "Intersheetrefs" "${INTERSHEET_REFS}"
-			(at 56.9467 120.65 0)
+			(at 55.9791 120.65 0)
 			(effects
 				(font
@@
 		)
 	)
-	(global_label "D_D"
+	(global_label "D_LS"
 		(shape input)
 		(at 63.5 127 180)
@@
 		)
 		(property "Intersheetrefs" "${INTERSHEET_REFS}"
-			(at 57.0072 127 0)
+			(at 56.0396 127 0)
 			(effects
 				(font

Commit message: more documentation
Parts:
- removed U10, U11, U6, U8, U9: 74LS32, symbol 74xx:74LS32
- added U2: 4078, symbol 4xxx_IEEE:4078
Connections:
- net S: now also U2.1
- net at U1.3 (QA): now also U2.2
- net at U1.2 (QB): now also U2.3
- net at U1.6 (QC): now also U2.4
- net at U1.7 (QD): now also U2.5
- net at U13.2 (QB): now also U2.10
- net at U13.3 (QA): now also U2.9
- net at U13.6 (QC): now also U2.11
- net at U13.7 (QD): now also U2.12
- no-connect marks 10 -> 11

Commit message: more documentation
Connections:
- net S renamed SET_S
Changed lines of the file:
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@@
 		)
 	)
-	(global_label "S"
+	(global_label "SET_S"
 		(shape output)
 		(at 234.95 82.55 0)
@@
 		)
 		(property "Intersheetrefs" "${INTERSHEET_REFS}"
-			(at 239.1447 82.55 0)
+			(at 243.4384 82.55 0)
 			(effects
 				(font
