File: doc/circuits/control_unit.kicad_sch (KiCad schematic)
At the start: 14 parts, among them U1 28C64, U10 74LS173, U11 74LS173, U12 74LS173, U13 74LS173, U14 74LS173, U2 74LS157, U3 28C64, U4 28C64, U5 28C64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

Commit message: more documentation
Parts:
- added U15: 74LS04, symbol 74xx:74LS04
- added U16: 74LS161, symbol 74xx:74LS161
Connections:
- net ERR: now also U9.6 (Q3); no longer U9.4 (Q1)
- net GND: now also U16.10 (CET), U16.7 (CEP)
- net M_CLK: now also U16.2 (CP)
- net RESET: now also U16.1 (~{MR})
- net at U2.12 (Zd): now also U16.6 (D3)
- net at U2.4 (Za): now also U16.3 (D0)
- net at U2.7 (Zb): now also U16.4 (D1)
- net at U2.9 (Zc): now also U16.5 (D2)
- net AE renamed SET_A
- net DPR renamed CLR_DP
- net LD_F renamed LD_FA
- net LD_I renamed LD_FBI
- net LD_FBI: now also U15.1
- net VE renamed SET_V
- new net: U15.2, U16.9 (~{PE})
- new net CLR_K: U9.4 (Q1)
- no-connect marks 10 -> 7
Other:
- note added: "NIBBLE SELECT + REGISTER"
- note removed: "NIBBLE SELECT"

Commit message: document restructuring
Other:
- note added: "CONTROL UNIT"
Changed lines of the file:
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@@
+		)
+	)
+	(text "CONTROL UNIT"
+		(exclude_from_sim no)
+		(at 233.934 175.006 0)
+		(effects
+			(font
+				(size 4 4)
+			)
 		)
 	)
