File: doc/circuits/register_driver.kicad_sch (KiCad schematic)
At the start: 6 parts, among them U1 74LS138, U2 74LS138, U3 74LS04, U4 74LS86, U5 74LS08, U6 74LS00

Commit message: Updated schematics
Parts:
- removed U6: 74LS00, symbol 74xx:74LS00
- added U6, U7: 74LS08, symbol 74xx:74LS08
Connections:
- net at U3.4: now also U6.1, U7.2; no longer U5.3
- net at U2.6 (E3): now also U6.3
- net at U3.2: now also U7.1
- net at U1.6 (E3): now also U7.3
- new net: U5.3, U6.2

Commit message: documented data and datapointer registers
Parts:
- removed U3: 74LS04, symbol 74xx:74LS04
- removed U5, U6, U7: 74LS08, symbol 74xx:74LS08
- added U10, U11, U3, U5, U6, U7, U8, U9: 74LS00, symbol 74xx:74LS00
Connections:
- net CLK: now also U5.2
- net DEC: now also U3.1, U3.2
- net INC: now also U8.1, U8.2
- net at U2.6 (E3): now also U10.3
- net at U1.6 (E3): now also U7.3
- net at U4.3: now also U5.1
- new net: U10.1, U10.2, U6.3
- new net: U3.3, U6.1, U9.2
- new net: U11.3, U6.2
- new net: U11.1, U11.2, U5.3
- new net: U8.3, U9.1
- new net: U7.1, U7.2, U9.3

Commit message: more documentation
Parts:
- removed U10, U11, U3, U5, U6, U7, U8, U9: 74LS00, symbol 74xx:74LS00
- removed U4: 74LS86, symbol 74xx:74LS86
- added U3: 74LS04, symbol 74xx:74LS04
Connections:
- net DEC: now also U3.3
- net INC: now also U3.1
- net M_CLK: now reaches U2.6 (E3)
- net M_CLK: now also U1.6 (E3)
- net GND: no longer names the net of U2.4 (E1), U2.5 (E2)
- net GND: now also U3.4; no longer U1.4 (E1), U1.5 (E2)
- new net: U1.4 (E1), U1.5 (E2), U3.2

Commit message: implemented program slots and updated docs
Connections:
- net RS2: now also U1.3 (A2)
Changed lines of the file:
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@@
+	)
+	(junction
+		(at 133.35 85.09)
+		(diameter 0)
+		(color 0 0 0 0)
 	)
 	(junction
@@
 	(wire
 		(pts
+			(xy 133.35 85.09) (xy 143.51 85.09)
+		)
+		(stroke
+			(width 0)
+			(type default)
+		)
+	)
+	(wire
+		(pts
 			(xy 168.91 85.09) (xy 180.34 85.09)
 		)
@@
 	(wire
 		(pts
-			(xy 133.35 45.72) (xy 133.35 125.73)
+			(xy 133.35 45.72) (xy 133.35 85.09)
 		)
 		(stroke
@@
 		)
 		(stroke
+			(width 0)
+			(type default)
+		)
+	)
+	(wire
+		(pts
+			(xy 133.35 85.09) (xy 133.35 125.73)
+		)
+		(stroke
