File: doc/circuits/master_clock.kicad_sch (KiCad schematic)
At the start: 27 parts, among them SW1 SW_MEC_5G, SW2 SW_Nidec_CAS-120A1, SW3 SW_MEC_5G, U1 LM555xM, U10 74LS14, U11 74LS173, U12 74LS32, U2 LM555xM, U3 LM555xM, U4 74LS14, U5 74LS00, U6 74LS00, U7 74LS00, U8 74LS00, U9 74LS14

Commit message: documented master clock
Parts:
- added C6: 0.01uF, symbol Device:C
- added C7: 1uF, symbol Device:C
- added RA3: 1K, symbol Device:R
- added RA4: 470K, symbol Device:R
- added SW4: SW_MEC_5G, symbol Switch:SW_MEC_5G
- added U13: LM555xM, Package_SO:SOIC-8_3.9x4.9mm_P1.27mm, symbol Timer:LM555xM
- R3: value 10K -> 1K
Connections:
- net +5V: now also RA3.2, RA4.2
- net GND: now also C6.1, C7.2, SW4.1 (A), SW4.2 (A)
- net RESET: now also U13.3 (Q)
- new net: RA3.1, SW4.3 (B), SW4.4 (B), U13.2 (TR)
- new net: C7.1, RA4.1, U13.6 (THR), U13.7 (DIS)
- new net: C6.2, U13.5 (CV)
- no-connect marks 5 -> 6
Other:
- note added: "RESET"
- company: (none) -> J. Heit

Commit message: More documentation done
Parts:
- removed C1: 1uF, symbol Device:C
- removed FREQ: 1M, symbol Device:R_Variable
- removed RA1: 1K, symbol Device:R
- added C8: 1uF, symbol Device:C
- added C9: 0.1uF, symbol Device:C
- added FREQ1: 1M, symbol Device:R_Variable
- added RA5: 1K, symbol Device:R
- added RA6: 100, symbol Device:R
- added SW5: SW_DIP_x04, symbol Switch:SW_DIP_x04
Connections:
- net +5V: now also RA5.2, RA6.2
- net GND: now also C8.2, C9.2
- net at U1.7 (DIS): now also FREQ1.1, SW5.1, SW5.2
- net at U1.2 (TR), U1.6 (THR): now also FREQ1.2, SW5.3, SW5.4
- new net: C9.1, SW5.6
- new net: RA5.1, SW5.8
- new net: RA6.1, SW5.7
- new net: C8.1, SW5.5
Other:
- note added: "RC-TIME SELECT"

Commit message: more documentation
Parts:
- removed FREQ1: 1M, symbol Device:R_Variable
- removed RA6: 100, symbol Device:R
- removed SW3: SW_MEC_5G, symbol Switch:SW_MEC_5G
- removed SW5: SW_DIP_x04, symbol Switch:SW_DIP_x04
- removed U10, U4, U9: 74LS14, symbol 74xx:74LS14
- added C1, C12, C14, C15, C16: 0.1nF, symbol Device:C
- added C10: 0.01uF, symbol Device:C
- added C11: 1nF, symbol Device:C
- added C13: 10uF, symbol Device:C
- added C17: 4.7uF, symbol Device:C
- added R4: 2K, symbol Device:R
- added R5: 10K, symbol Device:R_Variable
- added R6, R7, R8: 1K, symbol Device:R
- added R9: 680K, symbol Device:R
- added SW3: SW_DIP_x06, symbol Switch:SW_DIP_x06
- added SW5: SW_MEC_5G, symbol Switch:SW_MEC_5G
- added U10, U15, U16: 74LS123, symbol 74xx:74LS123
- added U14, U4, U9: 74LS04, symbol 74xx:74LS04
- added U17: 74LS76, symbol 74xx:74LS76
Connections:
- net CLK is gone; now on net M_CLK: U11.7 (Cp)
- net +5V: now also R5.1, R6.1, R7.1, R8.1, R9.1, SW5.3 (B), SW5.4 (B), U10.11 (Clr), U10.3 (Clr), U16.3 (Clr), U17.16 (K), U17.2 (~{S}), U17.3 (~{R}), U17.4 (J); no longer RA5.2
- net GND: now also RA5.1, C1.2, C10.2, C11.2, C12.2, C13.2; no longer R3.2
- net M_CLK: now also U10.5 (Q)
- net at U1.7 (DIS): now also R4.1
- net at U1.2 (TR), U1.6 (THR): now also R3.1, C1.1, R4.2, SW3.10, SW3.11, SW3.12, SW3.7, SW3.8, SW3.9
- net at U11.3 (Q0): now also U9.1
- net at C9.1: now also SW3.3
- net at U3.3 (Q), U6.2: now also U14.1
- net at U5.2: now also U14.2
- net at U8.3: now also U4.1
- net at U12.1: now also U15.13 (Q), U16.2 (B); no longer R3.1
- net at U1.3 (Q): now also U17.1 (C); no longer U6.1
- net at U8.2: now also U9.2
- net at C8.1: now also SW3.2
- new net: C14.1, U10.14 (Cext)
- new net: C14.2, R6.2, U10.15 (RCext)
- new net: C17.2, R9.2, U16.15 (RCext)
- new net: C16.2, R8.2, U15.15 (RCext)
- new net: U17.15 (Q), U6.1
- new net: C13.1, SW3.1
- new net: C10.1, SW3.4
- new net: C11.1, SW3.5
- new net: C12.1, SW3.6
- new net: R3.2, R5.2
- new net: C15.1, U10.6 (Cext)
- new net: C15.2, R7.2, U10.7 (RCext)
- new net: U10.2 (B), U10.9 (A), U4.2
- new net: C16.1, U15.14 (Cext)
- new net: RA5.2, SW5.1 (A), SW5.2 (A), U15.2 (B)
- new net: C17.1, U16.14 (Cext)
- new net: U15.3 (Clr), U16.4 (~{Q})
- new net D_CLK: U10.13 (Q)
- no-connect marks 6 -> 15
Other:
- note added: "CLOCK SPLITTER"

Commit message: more doc
Parts:
- added C18: 20uF, symbol Device:C
- added R10: 22K, symbol Device:R
- added U18: 74LS32, symbol 74xx:74LS32
- added U19: 74LS14, symbol 74xx:74LS14
Connections:
- net +5V: now also R10.2
- net GND: now also C18.1
- net RESET: now also U18.3; no longer U12.2, U13.3 (Q)
- new net: C18.2, R10.1, U19.1
- new net: U12.2, U13.3 (Q), U18.2
- new net: U18.1, U19.2
Other:
- note added: "POR"
